Commit message: passive joints

File: turtlebot_arm_description/urdf/turtlebot_arm.urdf (robot description, URDF)
Before this commit: robot turtlebot_arm, 23 links, 23 joints
Links:
- added link plate_top_link
Joints:
- added joint wheel_left_joint: type fixed, parent plate_top_link, child arm_base_link
- added joint wheel_right_joint: type fixed, parent plate_top_link, child arm_base_link

File: turtlebot_arm_description/urdf/turtlebot_arm.urdf.xacro (robot description, xacro)
@@ -13,5 +13,4 @@
     <xacro:property name="wrist_llimit" value="-1.745"/>
     <xacro:property name="wrist_ulimit" value="1.745"/>
-    <xacro:macro params="parent">
     <!-- Included URDF Files -->
     <xacro:include filename="$(find turtlebot_arm_description)/urdf/turtlebot_arm.xacro"/>
@@ -19,5 +18,5 @@
     <!-- link name="base_link"/ -->
     <!-- Turtlebot arm macro -->
-    <turtlebot_arm parent="${parent}" color="Gray" gripper_color="Gray"
+    <turtlebot_arm parent="plate_top_link" color="Gray" gripper_color="Gray"
                     pincher_gripper="false" turtlebot_gripper="true">
       <!-- Place the "floating" arm at the location it should be if mounted on a turtlebot,
@@ -25,4 +24,3 @@
       <origin xyz="0.1 0 0.02" rpy="0 0 -1.57075"/>
     </turtlebot_arm>
-    </xacro:macro>
 </robot>

File: turtlebot_arm_description/urdf/turtlebot_arm.xacro (robot description, xacro)
@@ -16,12 +16,21 @@
   </material>
   <xacro:macro name="turtlebot_arm" params="parent color pincher_gripper turtlebot_gripper gripper_color *origin">
+    <link name="plate_top_link"/>
+    <joint name="wheel_left_joint" type="fixed">
+      <parent link="plate_top_link"/>
+      <child link="arm_base_link"/>
+    </joint>
+    <joint name="wheel_right_joint" type="fixed">
+      <parent link="plate_top_link"/>
+      <child link="arm_base_link"/>
+    </joint>
     <link name="arm_base_link"/>
     <joint name="arm_base_joint" type="fixed">
       <insert_block name="origin"/>
-      <parent link="${parent}"/>
+      <parent link="plate_top_link"/>
       <child link="arm_base_link"/>
     </joint>
     <!-- fake gripper_link joint gives us a free servo!
-         this makes us 5DOF and saves you $44.90
+         this makes us 5DOF and saves you $44.90f
          that's a lot of coin! >
     <link name="gripper_link"/>
@@ -32,5 +41,5 @@
       <limit effort="30" velocity="1" lower="-3.14" upper="3.14"/>
       <axis xyz="1 0 0"/>
-    </joint-->
+    </joint -->
     <!-- shoulder pan joint -->
     <dynamixel_AX12_fixed parent="arm_base_link" name="arm_shoulder_pan_servo">

Commit message: edits

File: turtlebot_arm_description/urdf/turtlebot_arm.urdf (robot description, URDF)
Before this commit: robot turtlebot_arm, 24 links, 25 joints
Links:
- added link gripper_link
Joints:
- removed joint wheel_left_joint
- removed joint wheel_right_joint
- added joint gripper_link_joint: type revolute, parent arm_wrist_flex_link, child gripper_link, origin xyz=0 0 0.112 rpy=0 -1.57 0, axis 1 0 0, limit lower=-3.14 upper=3.14 effort=30 velocity=1

File: turtlebot_arm_description/urdf/turtlebot_arm.xacro (robot description, xacro)
@@ -17,12 +17,5 @@
   <xacro:macro name="turtlebot_arm" params="parent color pincher_gripper turtlebot_gripper gripper_color *origin">
     <link name="plate_top_link"/>
-    <joint name="wheel_left_joint" type="fixed">
-      <parent link="plate_top_link"/>
-      <child link="arm_base_link"/>
-    </joint>
-    <joint name="wheel_right_joint" type="fixed">
-      <parent link="plate_top_link"/>
-      <child link="arm_base_link"/>
-    </joint>
+    <!-- link name="base_link" / -->
     <link name="arm_base_link"/>
     <joint name="arm_base_joint" type="fixed">
@@ -33,5 +26,5 @@
     <!-- fake gripper_link joint gives us a free servo!
          this makes us 5DOF and saves you $44.90f
-         that's a lot of coin! >
+         that's a lot of coin! -->
     <link name="gripper_link"/>
     <joint name="gripper_link_joint" type="revolute">
@@ -41,5 +34,5 @@
       <limit effort="30" velocity="1" lower="-3.14" upper="3.14"/>
       <axis xyz="1 0 0"/>
-    </joint -->
+    </joint>
     <!-- shoulder pan joint -->
     <dynamixel_AX12_fixed parent="arm_base_link" name="arm_shoulder_pan_servo">
